Commit message: update readme requirement panda

File: panda/panda_hand.urdf (robot description, URDF)
Before this commit: robot panda_hand, 4 links, 3 joints
Links:
- link panda_hand: geometry collision mesh filename=grasp/panda/franka_description/meshes/collision/hand.stl; visual mesh filename=grasp/panda/franka_description/meshes/visual/hand.dae
- link panda_leftfinger: geometry collision mesh filename=grasp/panda/franka_description/meshes/collision/finger.stl; visual mesh filename=grasp/panda/franka_description/meshes/visual/finger.dae
- link panda_rightfinger: geometry collision mesh filename=grasp/panda/franka_description/meshes/collision/finger.stl; visual mesh filename=grasp/panda/franka_description/meshes/visual/finger.dae
